File: hardware/pcb/playgrounds/ch9350/ch9350.kicad_sch (KiCad schematic)
At the start: 14 parts, among them J1 USB_C_Receptacle_USB2.0_16P, J2 USB_A_Stacked, J3 Conn_01x02_Pin, J4 Conn_01x02_Pin, J5 Conn_01x02_Pin, J6 Conn_01x02_Pin, J7 Conn_02x08_Odd_Even, SW1 SW_Push, SW2 SW_Push, SW4 SW_Push_Dual, U1 CH9350, U2 CH9350

Commit message: ch9350 devboard schematic
Parts:
- removed J3, J4, J5, J6: Conn_01x02_Pin, symbol Connector:Conn_01x02_Pin
- added D1, D2, D3, D4, D5, D6: 19-213/Y2C-CQ2R2L/3T(CY), LED_SMD:LED_0603_1608Metric, symbol Device:LED_Small
- added J3: Conn_02x04_Odd_Even, symbol Connector_Generic:Conn_02x08_Odd_Even
- added J5: Conn_02x08_Odd_Even, symbol Connector_Generic:Conn_02x10_Odd_Even
- added Q1, Q2, Q3, Q4, Q5, Q6: MMBT2222A, Package_TO_SOT_SMD:SOT-23, symbol Transistor_BJT:MMBT5550L
- added R10, R12, R14, R4, R6, R8: 6K2, symbol Device:R_Small
- added R11, R13, R3, R5, R7, R9: 1K, symbol Device:R_Small
- J4: renamed from J7; symbol Connector_Generic:Conn_02x08_Odd_Even -> Connector_Generic:Conn_02x10_Odd_Even
- renumbered SW4 to SW3
Connections:
- net RESET1 is gone; now on net RESETa: SW1.1
- net VDD1 is gone; now on net VDDa: SW1.2, SW3.2
- net VDD2 is gone; now on net VDDb: SW2.2, SW3.4
- net GND: now also J4.10 (Pin_10), J4.12 (Pin_12), J4.4 (Pin_4), J4.6 (Pin_6), J4.8 (Pin_8), J5.10 (Pin_10), J5.12 (Pin_12), J5.2 (Pin_2), J5.4 (Pin_4), J5.6 (Pin_6), J5.8 (Pin_8), Q1.1 (B), Q2.1 (B), Q3.1 (B), Q4.1 (B), Q5.1 (B), Q6.1 (B), R10.2, R11.2, R12.2, R13.2, R14.2, R3.2, R4.2, R5.2, R6.2, R7.2, R8.2, R9.2
- net RXDa: now also J3.13 (Pin_13)
- net RXDb: now also J3.16 (Pin_16)
- net TXDa: now also J3.15 (Pin_15)
- net TXDb: now also J3.14 (Pin_14)
- net VBUS: now also J3.2 (Pin_2), J3.4 (Pin_4)
- net VBUSa: now also J3.1 (Pin_1)
- net VBUSb: now also J3.3 (Pin_3)
- net xOSCa: now reaches J4.11 (Pin_11)
- net xOSCa: now also U1.6 (xOSC)
- net XIa: now reaches J4.13 (Pin_13)
- net XIa: now also U1.16 (XI)
- net XOa: now reaches J4.14 (Pin_14)
- net XOa: now also U1.17 (XO)
- net IO1a: now reaches J4.15 (Pin_15)
- net IO1a: now also U1.21 (IO1)
- net IO2a: now reaches J4.16 (Pin_16)
- net IO2a: now also U1.22 (IO2)
- net S0a: now reaches J4.3 (Pin_3)
- net S0a: now also U1.4 (S0)
- net S1a: now reaches J4.5 (Pin_5)
- net S1a: now also U1.5 (S1)
- net BAUD0a: now reaches J4.7 (Pin_7)
- net BAUD0a: now also U1.38 (BAUD0)
- net BAUD1a: now reaches J4.9 (Pin_9)
- net BAUD1a: now also U1.37 (BAUD1)
- net LED1a: now reaches U1.1 (LED1)
- net LED1a: now also D2.2 (A), R5.1
- net LED2a: now reaches U1.2 (LED2)
- net LED2a: now also D3.2 (A), R7.1
- net IO3a: now reaches U1.23 (IO3)
- net IO3a: now also J4.17 (Pin_17)
- net IO4a: now reaches U1.24 (IO4)
- net IO4a: now also J4.18 (Pin_18)
- net TNOWa: now reaches U1.26 (TNOW)
- net TNOWa: now also J4.19 (Pin_19)
- net VDDa: now reaches U1.42 (VDD33)
- net LED0a: now reaches U1.48 (LED0)
- net LED0a: now also D1.2 (A), R3.1
- net DEBUGa: now reaches U1.7 (DEBUG)
- net DEBUGa: now also J4.20 (Pin_20)
- net LED1b: now reaches U2.1 (LED1)
- net LED1b: now also D5.2 (A), R11.1
- net XIb: now reaches U2.16 (XI)
- net XIb: now also J5.13 (Pin_13)
- net XOb: now reaches U2.17 (XO)
- net XOb: now also J5.14 (Pin_14)
- net LED2b: now reaches U2.2 (LED2)
- net LED2b: now also D6.2 (A), R13.1
- net IO1b: now reaches U2.21 (IO1)
- net IO1b: now also J5.15 (Pin_15)
- net IO2b: now reaches U2.22 (IO2)
- net IO2b: now also J5.16 (Pin_16)
- net IO3b: now reaches U2.23 (IO3)
- net IO3b: now also J5.17 (Pin_17)
- net IO4b: now reaches U2.24 (IO4)
- net IO4b: now also J5.18 (Pin_18)
- net TNOWb: now reaches U2.26 (TNOW)
- net TNOWb: now also J5.19 (Pin_19)
- net BAUD1b: now reaches U2.37 (BAUD1)
- net BAUD1b: now also J5.9 (Pin_9)
- net BAUD0b: now reaches U2.38 (BAUD0)
- net BAUD0b: now also J5.7 (Pin_7)
- net S0b: now reaches U2.4 (S0)
- net S0b: now also J5.3 (Pin_3)
- net VDDb: now reaches U2.42 (VDD33)
- net SELb: now reaches U2.45 (SEL)
- net SELb: now also J5.1 (Pin_1)
- net LED0b: now reaches U2.48 (LED0)
- net LED0b: now also D4.2 (A), R9.1
- net S1b: now reaches U2.5 (S1)
- net S1b: now also J5.5 (Pin_5)
- net xOSCb: now reaches U2.6 (xOSC)
- net xOSCb: now also J5.11 (Pin_11)
- net DEBUGb: now reaches U2.7 (DEBUG)
- net DEBUGb: now also J5.20 (Pin_20)
- net RESET2 renamed RESETb
- net SEL1 renamed SELa
- new net: Q5.2 (E), R12.1
- new net: D5.1 (K), Q5.3 (C)
- new net: Q2.2 (E), R6.1
- new net: Q1.2 (E), R4.1
- new net: Q4.2 (E), R10.1
- new net: D4.1 (K), Q4.3 (C)
- new net: D1.1 (K), Q1.3 (C)
- new net: Q6.2 (E), R14.1
- new net: D6.1 (K), Q6.3 (C)
- new net: D2.1 (K), Q2.3 (C)
- new net: Q3.2 (E), R8.1
- new net: D3.1 (K), Q3.3 (C)
- no-connect marks 10 -> 12

Commit message: ch9350 devboard schematic
Connections:
- net GND: now also J2.8 (GND2); no longer J2.9 (Shield)
- net GNDPWR: now also J2.9 (Shield); no longer J2.8 (GND2)
- no-connect marks 12 -> 15
Other:
- moved on the sheet: J2
Changed lines of the file:
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@@
 	)
 	(junction
-		(at 256.54 144.78)
+		(at 269.24 144.78)
 		(diameter 0)
 		(color 0 0 0 0)
@@
 	)
 	(no_connect
+		(at 203.2 154.94)
+	)
+	(no_connect
 		(at 93.98 124.46)
 	)
@@
 	)
 	(no_connect
+		(at 226.06 144.78)
+	)
+	(no_connect
 		(at 93.98 129.54)
 	)
@@
 	)
 	(no_connect
+		(at 226.06 147.32)
+	)
+	(no_connect
 		(at 106.68 127)
 	)
@@
 	(wire
 		(pts
-			(xy 269.24 119.38) (xy 279.4 119.38)
+			(xy 261.62 119.38) (xy 251.46 119.38)
 		)
 		(stroke
@@
 	(wire
 		(pts
-			(xy 269.24 127) (xy 279.4 127)
+			(xy 261.62 127) (xy 251.46 127)
 		)
 		(stroke
@@
 	(wire
 		(pts
-			(xy 269.24 129.54) (xy 279.4 129.54)
+			(xy 261.62 129.54) (xy 251.46 129.54)
 		)
 		(stroke
@@
 	(wire
 		(pts
-			(xy 259.08 144.78) (xy 259.08 142.24)
+			(xy 271.78 144.78) (xy 271.78 142.24)
 		)
 		(stroke
@@
 	(wire
 		(pts
-			(xy 269.24 116.84) (xy 279.4 116.84)
+			(xy 261.62 116.84) (xy 251.46 116.84)
 		)
 		(stroke
@@
 	(wire
 		(pts
-			(xy 261.62 142.24) (xy 261.62 147.32)
+			(xy 274.32 142.24) (xy 274.32 147.32)
 		)
 		(stroke
@@
 	(wire
 		(pts
-			(xy 256.54 144.78) (xy 256.54 147.32)
+			(xy 269.24 144.78) (xy 269.24 147.32)
 		)
 		(stroke
@@
 	(wire
 		(pts
-			(xy 256.54 142.24) (xy 256.54 144.78)
+			(xy 269.24 142.24) (xy 269.24 144.78)
 		)
 		(stroke
@@
 	(wire
 		(pts
-			(xy 269.24 132.08) (xy 279.4 132.08)
+			(xy 261.62 132.08) (xy 251.46 132.08)
 		)
 		(stroke
@@
 	(wire
 		(pts
-			(xy 256.54 144.78) (xy 259.08 144.78)
+			(xy 269.24 144.78) (xy 271.78 144.78)
 		)
 		(stroke
@@
 	(wire
 		(pts
-			(xy 269.24 124.46) (xy 279.4 124.46)
+			(xy 261.62 124.46) (xy 251.46 124.46)
 		)
 		(stroke
@@
 	)
 	(label "DP2"
-		(at 279.4 129.54 180)
+		(at 251.46 129.54 0)
 		(fields_autoplaced yes)
 		(effects
@@
 				(size 1.27 1.27)
 			)
-			(justify right bottom)
+			(justify left bottom)
 		)
 	)
@@
 	)
 	(label "VBUS"
-		(at 279.4 116.84 180)
+		(at 251.46 116.84 0)
 		(fields_autoplaced yes)
 		(effects
@@
 				(size 1.27 1.27)
 			)
-			(justify right bottom)
+			(justify left bottom)
 		)
 	)
@@
 	)
 	(label "DP1"
-		(at 279.4 124.46 180)
+		(at 251.46 124.46 0)
 		(fields_autoplaced yes)
 		(effects
@@
 				(size 1.27 1.27)
 			)
-			(justify right bottom)
+			(justify left bottom)
 		)
 	)
@@
 	)
 	(label "VBUS"
-		(at 279.4 119.38 180)
+		(at 251.46 119.38 0)
 		(fields_autoplaced yes)
 		(effects
@@
 				(size 1.27 1.27)
 			)
-			(justify right bottom)
+			(justify left bottom)
 		)
 	)
@@
 	)
 	(label "DM2"
-		(at 279.4 132.08 180)
+		(at 251.46 132.08 0)
 		(fields_autoplaced yes)
 		(effects
@@
 				(size 1.27 1.27)
 			)
-			(justify right bottom)
+			(justify left bottom)
 		)
 	)
@@
 	)
 	(label "DM1"
-		(at 279.4 127 180)
+		(at 251.46 127 0)
 		(fields_autoplaced yes)
 		(effects
@@
 				(size 1.27 1.27)
 			)
-			(justify right bottom)
+			(justify left bottom)
 		)
 	)
@@
 	(symbol
 		(lib_id "Connector:USB_A_Stacked")
-		(at 259.08 127 0)
+		(at 271.78 127 0)
+		(mirror y)
 		(unit 1)
 		(exclude_from_sim no)
@@
 		(on_board yes)
 		(dnp no)
-		(fields_autoplaced yes)
 		(property "Reference" "J2"
-			(at 259.08 109.22 0)
+			(at 271.78 109.22 0)
 			(effects
 				(font
@@
 		)
 		(property "Value" "USB_A_Stacked"
-			(at 259.08 111.76 0)
+			(at 271.78 111.76 0)
 			(effects
 				(font
@@
 		)
 		(property "Footprint" ""
-			(at 262.89 140.97 0)
+			(at 267.97 140.97 0)
 			(effects
 				(font
@@
 		)
 		(property "Datasheet" " ~"
-			(at 264.16 125.73 0)
+			(at 266.7 125.73 0)
 			(effects
 				(font
@@
 		)
 		(property "Description" "USB Type A connector, stacked"
-			(at 259.08 127 0)
+			(at 271.78 127 0)
 			(effects
 				(font
@@
 	(symbol
 		(lib_id "power:GNDPWR")
-		(at 261.62 147.32 0)
+		(at 274.32 147.32 0)
 		(mirror y)
 		(unit 1)
@@
 		(fields_autoplaced yes)
 		(property "Reference" "#PWR06"
-			(at 261.62 152.4 0)
+			(at 274.32 152.4 0)
 			(effects
 				(font
@@
 		)
 		(property "Value" "GNDPWR"
-			(at 261.747 152.4 0)
+			(at 274.447 152.4 0)
 			(effects
 				(font
@@
 		)
 		(property "Footprint" ""
-			(at 261.62 148.59 0)
+			(at 274.32 148.59 0)
 			(effects
 				(font
@@
 		)
 		(property "Datasheet" ""
-			(at 261.62 148.59 0)
+			(at 274.32 148.59 0)
 			(effects
 				(font
@@
 		)
 		(property "Description" ""
-			(at 261.62 147.32 0)
+			(at 274.32 147.32 0)
 			(effects
 				(font
@@
 	(symbol
 		(lib_id "power:GND")
-		(at 256.54 147.32 0)
+		(at 269.24 147.32 0)
 		(unit 1)
 		(exclude_from_sim no)
@@
 		(fields_autoplaced yes)
 		(property "Reference" "#PWR05"
-			(at 256.54 153.67 0)
+			(at 269.24 153.67 0)
 			(effects
 				(font
@@
 		)
 		(property "Value" "GND"
-			(at 256.54 152.4 0)
+			(at 269.24 152.4 0)
 			(effects
 				(font
@@
 		)
 		(property "Footprint" ""
-			(at 256.54 147.32 0)
+			(at 269.24 147.32 0)
 			(effects
 				(font
@@
 		)
 		(property "Datasheet" ""
-			(at 256.54 147.32 0)
+			(at 269.24 147.32 0)
 			(effects
 				(font
@@
 		)
 		(property "Description" "Power symbol creates a global label with name \"GND\" , ground"
-			(at 256.54 147.32 0)
+			(at 269.24 147.32 0)
 			(effects
 				(font
